File: hw/upm.kicad_pcb (KiCad board)
At the start: 2 copper layers, 4 parts, among them U1 ATSAMD21E15B, U2 MIC23150-SYMT, U3 USB2512B, U4 PAC1934

Commit message: wip
Parts:
- added C1: C0402_12p_25Vdc_C0G_2, C0402, F.Cu at (112.8, 69.1)
- added C10: C0402_1u_6.3Vdc_X7R, C0402, F.Cu at (128.8, 65.3)
- added C11: C0402_1u_6.3Vdc_X7R, C0402, F.Cu at (126.8, 67.4)
- added C12: C0402_1u_6.3Vdc_X7R, C0402, F.Cu at (128.8, 66.4)
- added C13: C0402_1u_6.3Vdc_X7R, C0402, F.Cu at (130.9, 65.3)
- added C14: C0402_1u_6.3Vdc_X7R, C0402, F.Cu at (126.8, 68.5)
- added C15: C0402_1u_6.3Vdc_X7R, C0402, F.Cu at (128.8, 67.4)
- added C2: C0402_12p_25Vdc_C0G_2, C0402, F.Cu at (112.8, 70.2)
- added C3: C0402_100n_25Vdc_X7R, C0402, F.Cu at (114.8, 69.1)
- added C4: C0402_1u_6.3Vdc_X7R, C0402, F.Cu at (112.8, 71.2)
- added C5: C0402_1u_6.3Vdc_X7R, C0402, F.Cu at (114.8, 70.2)
- added C6: C0402_100n_25Vdc_X7R, C0402, F.Cu at (116.9, 69.1)
- added C7: C0402_1u_6.3Vdc_X7R, C0402, F.Cu at (112.8, 72.3)
- added C8: C0402_1u_6.3Vdc_X7R, C0402, F.Cu at (126.8, 65.3)
- added C9: C0402_1u_6.3Vdc_X7R, C0402, F.Cu at (126.8, 66.4)
- added J1: FTSH-105-01-F-DV-K, footprints:TFM-105-02-S-D-WT, F.Cu at (128.3, 55.9)
- added J2: USB_A_292303-1, USB_A_TH, F.Cu at (91.4, 57.1)
- added R1: R0402_100R, R0402, F.Cu at (114.6, 71.3)
- added R10: R0402_2k20, R0402, F.Cu at (130.3, 68.8)
- added R11: R0402_46k40, R0402, F.Cu at (132.3, 67.7)
- added R2: R0402_46k40, R0402, F.Cu at (116.7, 70.2)
- added R3: R0402_46k40, R0402, F.Cu at (116.3, 71.4)
- added R4: R0402_46k40, R0402, F.Cu at (118.3, 70.2)
- added R5: R0402_12k10, R0402, F.Cu at (130.7, 66.4)
- added R6: R0402_46k40, R0402, F.Cu at (132.7, 65.4)
- added R7: R0402_46k40, R0402, F.Cu at (128.6, 68.5)
- added R8: R0402_46k40, R0402, F.Cu at (130.7, 67.6)
- added R9: R0402_2k20, R0402, F.Cu at (132.3, 66.5)
- added U5: LP3470IM5X-3.08_NOPB, footprints:SOT-23-5, F.Cu at (112.5, 60.4)
- added U6: NCP380HSNAJAAT1G, footprints:TSOT-23-6, F.Cu at (100.0, 62.1)
- moved U4 35.9 mm to (113.5, 56.0)
- moved U2 28.2 mm to (106.7, 64.8)
- moved U1 25.0 mm to (107.8, 56.4)
- moved U3 23.8 mm to (101.3, 56.8)
Connections:
- net Net-(U3-Pad26) renamed /RST_N
- net Net-(U4-Pad1) renamed /PAC_ALERT_N
- U3 pad 10: Net-(U3-Pad10) -> P3V3
- U3 pad 11: Net-(U3-Pad11) -> GND
- U3 pad 13: Net-(U3-Pad13) -> P3V3
- U3 pad 15: Net-(U3-Pad15) -> P3V3
- U3 pad 17: Net-(U3-Pad17) -> P3V3
- U3 pad 23: Net-(U3-Pad23) -> P3V3
- U3 pad 29: Net-(U3-Pad29) -> P3V3
- U3 pad 36: Net-(U3-Pad36) -> P3V3
- U3 pad 37: Net-(U3-Pad37) -> GND
- U3 pad 5: Net-(U3-Pad5) -> P3V3
- U4 pad 15: Net-(U4-Pad15) -> P3V3
- U4 pad 16: Net-(U4-Pad16) -> /PAC_PWRDN_N
- U4 pad 2: Net-(U4-Pad2) -> P3V3
- U4 pad 3: Net-(U4-Pad3) -> GND
- U4 pad 4: Net-(U4-Pad4) -> /I2C_SCL
- U4 pad 5: Net-(U4-Pad5) -> /I2C_SDA
- U4 pad 6: Net-(U4-Pad6) -> GND

Commit message: wip
Parts:
- added C16: C0603_10u_10Vdc_X7R, C0603, F.Cu at (98.4, 75.6)
- added C17: C0402_1u_6.3Vdc_X7R, C0402, F.Cu at (102.2, 73.9)
- added C18: C0402_100n_25Vdc_X7R, C0402, F.Cu at (105.1, 72.5)
- added C19: C0402_1u_6.3Vdc_X7R, C0402, F.Cu at (100.9, 76.8)
- added C20: C0402_1u_6.3Vdc_X7R, C0402, F.Cu at (103.7, 74.9)
- added C21: C0603_10u_10Vdc_X7R, C0603, F.Cu at (115.0, 83.0)
- added C22: C0402_1u_6.3Vdc_X7R, C0402, F.Cu at (105.1, 73.6)
- added C23: C0603_10u_10Vdc_X7R, C0603, F.Cu at (98.4, 77.0)
- added C24: C0402_12p_25Vdc_C0G_2, C0402, F.Cu at (102.9, 76.8)
- added C25: C0402_12p_25Vdc_C0G_2, C0402, F.Cu at (105.8, 74.7)
- added C26: C0603_10u_10Vdc_X7R, C0603, F.Cu at (101.3, 75.6)
- added L1: IHLP1212_1u_1, IHLP1212, F.Cu at (111.0, 80.0)
- added R12: R0402_100R, R0402, F.Cu at (106.9, 72.6)
- added R13: R0402_46k40, R0402, F.Cu at (104.8, 76.1)
- moved U2 17.4 mm to (115.0, 80.0)
Connections:
- net Net-(U1-Pad23) renamed /UC_USB_D_N
- U1 pad 1: Net-(U1-Pad1) -> /I2C_SDA
- U1 pad 10: Net-(U1-Pad10) -> GND
- U1 pad 2: Net-(U1-Pad2) -> /I2C_SCL
- U1 pad 24: Net-(U1-Pad24) -> /UC_USB_D_P
- U1 pad 26: Net-(U1-Pad26) -> /RST_N
- U1 pad 28: Net-(U1-Pad28) -> GND
- U1 pad 3: Net-(U1-Pad3) -> /PAC_ALERT_N
- U1 pad 30: Net-(U1-Pad30) -> P3V3
- U1 pad 33: Net-(U1-Pad33) -> GND
- U1 pad 4: Net-(U1-Pad4) -> /PAC_PWRDN_N
- U1 pad 9: Net-(U1-Pad9) -> P3V3
- U2 pad 1: Net-(U2-Pad1) -> Net-(L1-Pad1)
- U2 pad 2: Net-(U2-Pad2) -> Net-(L1-Pad1)
- U2 pad 3: Net-(U2-Pad3) -> Net-(C16-Pad1)
- U2 pad 4: Net-(U2-Pad4) -> P3V3
- U2 pad 5: Net-(U2-Pad5) -> GND
- U2 pad 6: Net-(U2-Pad6) -> Net-(C16-Pad1)
- U2 pad 7: Net-(U2-Pad7) -> Net-(C16-Pad1)
- U2 pad 8: Net-(U2-Pad8) -> GND
- U3 pad 3: Net-(U3-Pad3) -> /UC_USB_D_P
- U3 pad 4: Net-(U3-Pad4) -> /UC_USB_D_P
- U5 pad 2: Net-(U5-Pad2) -> GND
- U5 pad 3: Net-(U5-Pad3) -> P3V3
- U5 pad 4: Net-(U5-Pad4) -> P3V3
- U5 pad 5: Net-(U5-Pad5) -> /RST_N

Commit message: wip
Parts:
- added C27: C0402_1u_6.3Vdc_X7R, C0402, F.Cu at (103.9, 107.8)
- added C29: C0603_22n_100Vdc_X7R, C0603, F.Cu at (113.5, 101.0)
- added C30: C0603_22n_100Vdc_X7R, C0603, F.Cu at (113.5, 102.4)
- added C31: C0603_22n_100Vdc_X7R, C0603, F.Cu at (113.5, 103.7)
- added J3: DX4R005JJ2R1800, footprints:USB_Micro-B, F.Cu at (153.7, 58.4)
- added R14: R0402_46k40, R0402, F.Cu at (115.8, 100.9)
- added R15: R0402_46k40, R0402, F.Cu at (105.7, 107.8)
- added R16: R0402_21k, R0402, F.Cu at (115.8, 102.1)
- added R17: R0603_200R, R0603, F.Cu at (113.4, 105.1)
- added R18: R0603_51R, R0603, F.Cu at (113.4, 106.6)
- added R19: R0603_51R, R0603, F.Cu at (115.9, 105.1)
- added R20: R0603_51R, R0603, F.Cu at (115.9, 106.6)
- J2: footprint USB_A_TH -> footprints:USB_A_TH
- moved J1 37.2 mm to (91.4, 61.0), turned to 90 degrees
- moved J2 6.35 mm to (85.1, 57.2)
Connections:
- C16 pad 1: Net-(C16-Pad1) -> P5V0
- J2 pad 1: Net-(J2-Pad1) -> /DUT_USB_VBUS
- J2 pad 2: Net-(J2-Pad2) -> /DUT_USB_D_N
- J2 pad 3: Net-(J2-Pad3) -> /DUT_USB_D_P
- J2 pad 4: Net-(J2-Pad4) -> GND
- J2 pad 5: Net-(J2-Pad5) -> GND
- J2 pad 6: Net-(J2-Pad6) -> GND
- R2 pad 2: Net-(R2-Pad2) -> P5V0
- U1 pad 5: Net-(U1-Pad5) -> /DUT_USB_EN
- U1 pad 6: Net-(U1-Pad6) -> /DUT_USB_FLAG_N
- U2 pad 3: Net-(C16-Pad1) -> P5V0
- U2 pad 6: Net-(C16-Pad1) -> P5V0
- U2 pad 7: Net-(C16-Pad1) -> P5V0
- U3 pad 1: Net-(U3-Pad1) -> /DUT_USB_D_N
- U3 pad 2: Net-(U3-Pad2) -> /DUT_USB_D_P
- U6 pad 1: Net-(U6-Pad1) -> P5V0
- U6 pad 2: Net-(U6-Pad2) -> GND
- U6 pad 3: Net-(U6-Pad3) -> /DUT_USB_EN
- U6 pad 4: Net-(U6-Pad4) -> /DUT_USB_FLAG_N
- U6 pad 6: Net-(U6-Pad6) -> /DUT_USB_VBUS
Other:
- copper layers 2 -> 4

Commit message: R1 release of HW
Parts:
- added C28: PCAP_120u_4, footprints:CP_Elec_6.3x5.8, F.Cu at (135.2, 93.2)
- added FB1: BL0603_BLM18BB121SN1D, L0603, F.Cu at (167.4, 101.0)
- added J4: TFM-105-02-S-D-WT, TFM-105-02-S-D-WT, F.Cu at (137.3, 103.8)
- added Q1: PUMH13, footprints:SOT-363_SC-70-6, F.Cu at (145.8, 102.7)
- added Q2: PUMH13, footprints:SOT-363_SC-70-6, F.Cu at (145.8, 105.7)
- added R21: R0402_1k, R0402, F.Cu at (155.2, 100.6)
- added R22: R0805_0R1, R0805, F.Cu at (142.9, 90.5)
- added R23: R0402_46k40, R0402, F.Cu at (153.1, 93.8)
- added U7: USBLC6-4, SOT-23-6, F.Cu at (166.8, 97.4)
- added U8: USBLC6-4, SOT-23-6, F.Cu at (132.4, 98.6)
- added X1: NX2520SA-24.000000MHZ, NX2520SA, F.Cu at (166.1, 92.8)
- added X2: NX2520SA-16.000000MHZ, NX2520SA, F.Cu at (153.3, 103.9)
- J1: footprint footprints:TFM-105-02-S-D-WT -> footprints:FTSH-105-01-F-DV-K
- J3: footprint footprints:USB_Micro-B -> USB_Micro-B
- moved J1 80.1 mm to (159.4, 103.4), turned to 0 degrees
- moved C17 77.0 mm to (173.0, 104.2), turned to 270 degrees
- moved C16 74.0 mm to (167.4, 102.4), turned to 180 degrees
- moved C18 73.9 mm to (170.6, 106.7), turned to 180 degrees
- moved U5 73.0 mm to (170.6, 104.6), turned to 180 degrees
- moved U3 70.0 mm to (159.7, 95.5), turned to 270 degrees
- moved C1 60.6 mm to (167.6, 95.0)
- moved U1 60.6 mm to (151.5, 98.4)
- moved J2 60.4 mm to (129.0, 98.6)
- moved C4 60.2 mm to (168.9, 93.0)
- moved C24 59.1 mm to (155.2, 104.5), turned to 270 degrees
- moved L1 58.9 mm to (164.5, 104.7), turned to 90 degrees
- moved C26 58.5 mm to (157.7, 91.1)
- moved U2 58.1 mm to (167.4, 105.0), turned to 90 degrees
- moved U6 57.5 mm to (149.5, 91.3), turned to 180 degrees
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Connections:
- net Net-(C19-Pad1) renamed /VDDCORE
- net Net-(C25-Pad1) renamed /XTAL_IN
- net Net-(J3-Pad2) renamed /USB_D_N
- net Net-(J3-Pad3) renamed /USB_D_P
- net Net-(R12-Pad2) renamed /XTAL_OUT
- J1 pad 1: Net-(J1-Pad1) -> P3V3
- J1 pad 10: Net-(J1-Pad10) -> /RST_N
- J1 pad 2: Net-(J1-Pad2) -> /SWDIO
- J1 pad 3: Net-(J1-Pad3) -> GND
- J1 pad 4: Net-(J1-Pad4) -> /SWCLK
- J1 pad 5: Net-(J1-Pad5) -> GND
- J1 pad 6: Net-(J1-Pad6) -> /SWO
- J1 pad 9: Net-(J1-Pad9) -> GND
- R17 pad 1: /DUT_USB_VBUS -> Net-(R17-Pad1)
- U1 pad 11: Net-(Q2-Pad5) -> /OUT3_EN
- U1 pad 12: Net-(U1-Pad12) -> /DUT_DISCHARGE
- U1 pad 27: Net-(U1-Pad27) -> /SWO
- U1 pad 31: Net-(U1-Pad31) -> /SWCLK
- U1 pad 32: Net-(U1-Pad32) -> /SWDIO
- U1 pad 7: Net-(Q1-Pad5) -> /OUT1_EN
- U1 pad 8: Net-(Q2-Pad2) -> /OUT2_EN
- U3 pad 3: /UC_USB_D_P -> /UC_USB_D_N
- U4 pad 10: Net-(U4-Pad10) -> /SNS4_P
- U4 pad 11: Net-(U4-Pad11) -> Net-(R17-Pad1)
- U4 pad 12: Net-(U4-Pad12) -> /DUT_USB_VBUS
- U4 pad 13: Net-(U4-Pad13) -> /SNS2_P
- U4 pad 14: Net-(U4-Pad14) -> /SNS2_N
- U4 pad 7: Net-(U4-Pad7) -> /SNS3_N
- U4 pad 8: Net-(U4-Pad8) -> /SNS3_P
- U4 pad 9: Net-(U4-Pad9) -> /SNS4_N
- U6 pad 6: /DUT_USB_VBUS -> Net-(R17-Pad1)
Routing:
- net GND: track 0.00 -> 64.7 mm, vias 0 -> 64
- net P5V0: track 0.00 -> 48.1 mm, vias 0 -> 8
- net /DUT_USB_D_N: track 0.00 -> 45.3 mm, vias 0 -> 2
- net /DUT_USB_D_P: track 0.00 -> 45.3 mm, vias 0 -> 2
- net /DUT_USB_VBUS: track 0.00 -> 42.2 mm, vias 0 -> 1
- net /RST_N: track 0.00 -> 39.9 mm, vias 0 -> 3
- net P3V3: track 0.00 -> 33.9 mm, vias 0 -> 34
- net /SNS4_N: track 0.00 -> 32.3 mm, vias 0 -> 2
- net /SNS4_P: track 0.00 -> 28.8 mm, vias 0 -> 2
- net /SWCLK: track 0.00 -> 22.4 mm, vias 0 -> 3
- net /SNS3_P: track 0.00 -> 22.1 mm, vias 0 -> 2
- net /SNS3_N: track 0.00 -> 21.6 mm, vias 0 -> 2
- net /SNS2_P: track 0.00 -> 20.0 mm, vias 0 -> 2
- net /SWDIO: track 0.00 -> 17.1 mm, vias 0 -> 2
- net /SNS2_N: track 0.00 -> 16.3 mm, vias 0 -> 2
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- added copper zone on B.Cu, net GND
- added copper zone on F.Cu, net GND
- added copper zone on In1.Cu, net GND
- added copper zone on In2.Cu, net P3V3
Other:
- board outline added: 58 x 18 mm
- net class Default: clearance 0.2 -> 0.127; trace_width 0.25 -> 0.127; via_dia 0.8 -> 0.45; via_drill 0.4 -> 0.254
- rule pad_to_mask_clearance: 0.2 -> 0.05
- rule trace_clearance: 0.2 -> 0.127
- rule trace_min: 0.2 -> 0.127
- rule via_min_drill: 0.3 -> 0.254
- rule via_min_size: 0.4 -> 0.45
- board text added: "JOP 2018"
- board text added: "UPM R1"
