File: hw/upm.sch (KiCad schematic (older format))
At the start: 8 parts, among them J1 FTSH-105-01-F-DV-K, J2 USB_A_292303-1, U1 ATSAMD21E15B, U2 MIC23150-SYMT, U3 USB2512B, U4 PAC1934, U5 LP3470M5-3.08, U6 NCP380HSNAJAAT1G

Commit message: wip
Parts:
- removed U5: LP3470M5-3.08, symbol power:LP3470M5-3.08
- added C1, C2: C0402_12p_25Vdc_C0G_2, C0402, symbol capacitors_murata_GRM:C0402_12p_25Vdc_C0G_2
- added C10, C11, C12, C13, C14, C15, C4, C5, C7, C8, C9: C0402_1u_6.3Vdc_X7R, C0402, symbol capacitors_murata_GRM:C0402_1u_6.3Vdc_X7R
- added C3, C6: C0402_100n_25Vdc_X7R, C0402, symbol capacitors_murata_GRM:C0402_100n_25Vdc_X7R
- added R1: R0402_100R, R0402, symbol vishay_resistors:R0402_100R
- added R10, R9: R0402_2k20, R0402, symbol vishay_resistors:R0402_2k20
- added R11, R2, R3, R4, R6, R7, R8: R0402_46k40, R0402, symbol vishay_resistors:R0402_46k40
- added R5: R0402_12k10, R0402, symbol vishay_resistors:R0402_12k10
- added U5: LP3470IM5X-3.08_NOPB, footprints:SOT-23-5, symbol power:LP3470IM5X-3.08_NOPB
- added U7, U8: USBLC6-4, TO_SOT_Packages_SMD:SOT-23-6, symbol esd:USBLC6-4
- added X1: NX2520SA-24.000000MHZ, NX2520SA, symbol xtal_NDK:NX2520SA-24.000000MHZ
- added X2: NX2520SA-16.000000MHZ, NX2520SA, symbol xtal_NDK:NX2520SA-16.000000MHZ
- J1: footprint Jonas:FTSH-105-01-F-DV-K -> footprints:TFM-105-02-S-D-WT
- J2: footprint (none) -> USB_A_TH
- U6: footprint (none) -> footprints:TSOT-23-6; Manufacturer (none) -> ONSemi; Part Number (none) -> NCP380HSNAJAAT1G
Connections:
- net labels added: GND, I2C_SCL, I2C_SDA, P3V3, PAC_ALERT_N, PAC_PWRDN_N, RST_N
- wire segments 0 -> 138
- no-connect marks 0 -> 2

Commit message: wip
Parts:
- added C16, C21, C23, C26: C0603_10u_10Vdc_X7R, C0603, symbol capacitors_murata_GRM:C0603_10u_10Vdc_X7R
- added C17, C19, C20, C22: C0402_1u_6.3Vdc_X7R, C0402, symbol capacitors_murata_GRM:C0402_1u_6.3Vdc_X7R
- added C18: C0402_100n_25Vdc_X7R, C0402, symbol capacitors_murata_GRM:C0402_100n_25Vdc_X7R
- added C24, C25: C0402_12p_25Vdc_C0G_2, C0402, symbol capacitors_murata_GRM:C0402_12p_25Vdc_C0G_2
- added L1: IHLP1212_1u_1, IHLP1212, symbol vishay_IHLP_inductors:IHLP1212_1u_1
- added R12: R0402_100R, R0402, symbol vishay_resistors:R0402_100R
- added R13: R0402_46k40, R0402, symbol vishay_resistors:R0402_46k40
Connections:
- net labels added: UC_USB_D_N, UC_USB_D_P
- wire segments 138 -> 226

Commit message: wip
Parts:
- added C27: C0402_1u_6.3Vdc_X7R, C0402, symbol capacitors_murata_GRM:C0402_1u_6.3Vdc_X7R
- added C28: PCAP_120u_4, PCAP_6.60, symbol nichicon_polymer_cap:PCAP_120u_4
- added C29, C30, C31: C0603_22n_100Vdc_X7R, C0603, symbol capacitors_murata_GRM:C0603_22n_100Vdc_X7R
- added FB1: BL0603_BLM18BB121SN1D, L0603, symbol beads_BLM:BL0603_BLM18BB121SN1D
- added J3: DX4R005JJ2R1800, USB_Micro-B, symbol connectors:DX4R005JJ2R1800
- added Q1, Q2: PUMH13, TO_SOT_Packages_SMD:SC-70-6, symbol transistors:PUMH13
- added R14, R15: R0402_46k40, R0402, symbol vishay_resistors:R0402_46k40
- added R16: R0402_21k, R0402, symbol vishay_resistors:R0402_21k
- added R17: R0603_200R, R0603, symbol vishay_resistors:R0603_200R
- added R18, R19, R20: R0603_51R, R0603, symbol vishay_resistors:R0603_51R
Connections:
- net labels added: DUT_USB_D_N, DUT_USB_D_P, DUT_USB_EN, DUT_USB_FLAG_N, DUT_USB_VBUS, P5V0
- wire segments 226 -> 342
- no-connect marks 2 -> 7

Commit message: R1 release of HW
Parts:
- added J4: TFM-105-02-S-D-WT, TFM-105-02-S-D-WT, symbol connectors:TFM-105-02-S-D-WT
- added R21: R0402_1k, R0402, symbol vishay_resistors:R0402_1k
- added R22: R0805_0R1, R0805, symbol resistors_misc:R0805_0R1
- added R23: R0402_46k40, R0402, symbol vishay_resistors:R0402_46k40
- C28: footprint PCAP_6.60 -> footprints:CP_Elec_6.3x5.8
- J1: footprint footprints:TFM-105-02-S-D-WT -> footprints:FTSH-105-01-F-DV-K
- Q1, Q2: footprint TO_SOT_Packages_SMD:SC-70-6 -> footprints:SOT-363_SC-70-6; Manufacturer (none) -> Nexperia; Part Number (none) -> PUMH13,115
- U7, U8: footprint TO_SOT_Packages_SMD:SOT-23-6 -> SOT-23-6
Connections:
- net labels added: DUT_DISCHARGE, OUT1_EN, OUT2_EN, OUT3_EN, SNS2_N, SNS2_P, SNS3_N, SNS3_P, SNS4_N, SNS4_P, SWCLK, SWDIO, SWO, USB_D_N, USB_D_P, VDDCORE, XTAL_IN, XTAL_OUT
- wire segments 342 -> 389
- no-connect marks 7 -> 11
